File: 750 LFO S&H NOISE SLEW.sch (KiCad schematic (older format))
At the start: 158 parts

Commit message: working on 150 LFO
Parts:
- added C?: 100n, MyModules:SM0603-C-JRL, symbol C_US
- added C?: 47n, MyModules:SM0603-C-JRL, symbol C_US
- added C?: 10p, MyModules:SM0603-C-JRL, symbol C_US
- added D? (x3): 1N4148, MyModules:SOD323-JRL, symbol DIODE
- added J?: JACK_MONO_SW, MyModules:PJ-301B-JACK-SLOTS, symbol JACK_MONO_SW
- added Q? (x2): DMMT3904W, MyModules:SOT363-JRL, symbol DMMT3904W
- added Q?: MMBT3904, SOT-23, symbol MMBT3904
- added R?: 22K, MyModules:SM0603-R-JRL, symbol R_US
- added R? (x3): 1K, MyModules:SM0603-R-JRL, symbol R_US
- added R?: 15K, MyModules:SM0603-R-JRL, symbol R_US
- added R? (x7): 10K, MyModules:SM0603-R-JRL, symbol R_US
- added R? (x2): 47K, MyModules:SM0603-R-JRL, symbol R_US
- added R?: 33K, MyModules:SM0603-R-JRL, symbol R_US
- added R? (x3): 100K, MyModules:SM0603-R-JRL, symbol R_US
- added R?: 180K, MyModules:SM0603-R-JRL, symbol R_US
- added U? (x2): TL072-, MyModules:TSSOP8-JRL, symbol TL072-
- added VR?: 100K, MyModules:RV09AF-40-ALPHA-POT, symbol POT_US
Connections:
- net +12V: now also Q?.2 (D), Q?.3 (C), R?.1, U?.8 (V+)
- net -12V: now also D?.1 (A), Q?.2 (E), Q?.5 (E), R?.2, R?.2, U?.4 (V-)
- net GND: now also C?.2, D?.1 (A), D?.2 (K), J?.1, Q?.4 (E), R?.2, R?.2, R?.2, R?.2
- net LFO_SINE: now also R?.2
- net WHITE_NOISE: now also C?.1; no longer C?.2
- net at R?.1, R?.2, U?.2 (-): now also C?.2; no longer C?.1
- net at U?.1: now also R?.1, R?.2
- net at U?.3 (+): now also R?.1, R?.1
- net at U?.4 (-): now also R?.1
- net at U?.5: now also Q?.3 (G), C?.1
- net at Q?.1 (S): now also R?.1, R?.1, R?.1
- net at Q?.3 (C): now also R?.1
- new net: R?.2, R?.2, U?.1
- new net: R?.2, R?.2, U?.2 (-)
- new net: R?.1, R?.1, U?.3 (+)
- new net: D?.1 (A), D?.2 (K), R?.2, U?.5 (+)
- new net: C?.2, R?.1, R?.1, U?.6 (-)
- new net: C?.1, R?.1, R?.2, U?.7
- new net: R?.2, VR?.2
- new net: Q?.3 (C), R?.2
- new net: Q?.2 (B), R?.2
- new net: C?.1, D?.2 (K), Q?.1 (B), Q?.1 (B), R?.1
- new net: Q?.6 (C), R?.1, R?.2
- new net: J?.3, R?.1
- new net: Q?.3 (C), R?.1
- new net: C?.2, R?.2
- no-connect marks 10 -> 12
Other:
- note added: "RAMP ADJUST"
- note added: "RESET"
- moved on the sheet: J?, Q?, R?, U?A, VR?

Commit message: schematic more or less captured. Still need to check and also confirm noise circuit
Parts:
- added C?: 100n, MyModules:SM0603-C-JRL, symbol C_US
- added C?: 4.7μ, symbol CP_US
- added D? (x3): 1N4148, MyModules:SOD323-JRL, symbol DIODE
- added D?: LED, MyModules:3MM-LED-C1A2, symbol LED
- added J?: JACK_MONO_SW, MyModules:PJ-301B-JACK-SLOTS, symbol JACK_MONO_SW
- added P? (x2): CONN_02X01, symbol CONN_02X01
- added Q?: MMBT3904, MyModules:SOT23-132-JRL, symbol MMBT3904
- added Q? (x2): J112, MyModules:SOT23-JRL, symbol Q_NJFET_SDG-RESCUE-Eurorack-JP6-filter
- added Q?: MMBT3904, SOT-23, symbol MMBT3904
- added Q?: MMBT3906, SOT-23, symbol MMBT3906
- added R? (x7): 100K, MyModules:SM0603-R-JRL, symbol R_US
- added R? (x2): 82K, MyModules:SM0603-R-JRL, symbol R_US
- added R? (x6): 1K, MyModules:SM0603-R-JRL, symbol R_US
- added R? (x4): 47K, MyModules:SM0603-R-JRL, symbol R_US
- added R? (x3): 39K, MyModules:SM0603-R-JRL, symbol R_US
- added R?: 15K, MyModules:SM0603-R-JRL, symbol R_US
- added R? (x2): 330K, MyModules:SM0603-R-JRL, symbol R_US
- added R?: 56K, MyModules:SM0603-R-JRL, symbol R_US
- added R?: 150K, MyModules:SM0603-R-JRL, symbol R_US
- added R?: 4.7K, MyModules:SM0603-R-JRL, symbol R_US
- added R?: 33K, MyModules:SM0603-R-JRL, symbol R_US
- added R?: 22K, MyModules:SM0603-R-JRL, symbol R_US
- added U? (x4): TL072-, MyModules:TSSOP8-JRL, symbol TL072-
- added U?: LM13700, MyModules:SO16-JRL, symbol LM13700
- added VR?: 1meg, MyModules:RV09AF-40-ALPHA-POT, symbol POT_US
- added VR?: 100K, MyModules:RV09AF-40-ALPHA-POT, symbol POT_US
- C?: value 10p -> 100n
Connections:
- net +12V: now also Q?.2 (D), Q?.3 (C), U?.8 (V+), U?.8 (V+), VR?.3, VR?.3
- net -12V: now also D?.1 (A), R?.2, R?.2, R?.2, R?.2, U?.4 (V-), U?.4 (V-), VR?.1
- net GND: now also D?.1 (K), J?.1, P?.1 (P1), Q?.1 (B), Q?.1 (S), R?.2, R?.2, R?.2, R?.2, R?.2, R?.2, R?.2, U?.5 (+)
- net LFO: now also R?.2
- net LFO_PULSE: now also D?.2 (K), R?.1, R?.1
- net LFO_RAMP: now also R?.2
- net LFO_TRI: now also R?.2
- net S&H_TRI: now also R?.1; no longer C?.2, R?.1, U?.7
- net at Q?.1 (S), R?.1, R?.1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: now also R?.1, R?.1
- net at R?.2, R?.2, U?.1: now also R?.1, D?.2 (K), R?.1
- net at VR?.3: now also R?.1, R?.2, U?.2 (-)
- net at J?.2: now also P?.2 (P2)
- net at J?.3, R?.1: now also P?.1 (P1)
- new net: C?.2, R?.1, R?.2, U?.7
- new net: C?.1, D?.2 (K), Q?.1 (B), R?.1
- new net: C?.2, P?.2 (P2)
- new net: R?.1, R?.2, U?.6 (-)
- new net: D?.1 (A), R?.1, R?.2, U?.7
- new net: Q?.1 (B), R?.2
- new net: Q?.2 (E), R?.1
- new net: D?.2 (A), R?.2
- new net: R?.1, R?.2, U?.1
- new net: Q?.2 (D), R?.2, U?.3 (+)
- new net: R?.1, R?.1, R?.1, R?.2, R?.2
- new net: D?.1 (A), Q?.3 (G), R?.1
- new net: R?.1, R?.1, R?.2, U?.6 (-)
- new net: R?.1, U?.5 (+)
- new net: R?.1, R?.2, U?.7
- new net: C?.2 (-), Q?.2 (E), R?.1
- new net: C?.1 (+), Q?.3 (C), Q?.3 (G), VR?.1, VR?.2
- new net: Q?.1 (S), R?.1, R?.1
- new net: Q?.2 (E), R?.2, R?.2
- new net: Q?.3 (C), R?.1
- new net: R?.1, VR?.2
- new net: R?.1, U?.1, U?.2 (-)
- new net: R?.1, U?.3 (+), U?.5
- new net: R?.2, U?.1
- new net: R?.1, R?.1, U?.3 (+)
- new net: R?.1, U?.4 (-)
- new net: J?.3, R?.2
Other:
- note added: "LEVEL"
- note added: "LFO OUT"
- note added: "NOT SURE HOW TO HANDLE\nRESET/GATE INPUT SO ADD\nJUMPERS FOR LFO RESET \nAND GATE DELAY INPUTS"
- note removed: "NEED TO TEST THIS\nLED CONFIGURATION"
- moved on the sheet: C?, D?, J?, P?, Q?, Q?A, Q?B, R?, SW?, TP?, U?, U?A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

Commit message: tidy up a bit. Could start part assignment and rough layout now
Parts:
- added TP? (x2): CONN_1, MyModules:TEST_POINT_LOOP_4592, symbol CONN_1
Connections:
- net at C?.1, J?.3, R?.1: now also TP?.1
- net at C?.2, R?.1, R?.2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: now also TP?.1
Other:
- moved on the sheet: D?, J?, R?, U?A

Commit message: noise source done. removed redundant power-on-reset circuit
Parts:
- removed C? (x2): 10μ, MyModules:2MM-POL-CAP, symbol CP_US
- removed C?: 100n, MyModules:SM0603-C-JRL, symbol C_US
- removed C?: 10p, MyModules:SM0603-C-JRL, symbol C_US
- removed C?: 39n, MyModules:SM0603-C-JRL, symbol C_US
- removed C?: 18n, MyModules:SM0603-C-JRL, symbol C_US
- removed C?: 0.47μ, MyModules:SM0603-C-JRL, symbol C_US
- removed D?: 1N914, MyModules:SOD323-C1A2, symbol D
- removed Q? (x2): DMMT3904W, MyModules:SOT363-JRL, symbol DMMT3904W
- removed R?: 100K, MyModules:SM0603-R-JRL, symbol R_US
- removed R?: 1K, MyModules:SM0603-R-JRL, symbol R_US
- removed R?: 680K, MyModules:SM0603-R-JRL, symbol R_US
- removed R?: 4.7K, MyModules:SM0603-R-JRL, symbol R_US
- removed R?: 15K, MyModules:SM0603-R-JRL, symbol R_US
- removed R? (x2): 22K, MyModules:SM0603-R-JRL, symbol R_US
- removed R?: 33K, MyModules:SM0603-R-JRL, symbol R_US
- removed R?: 330, MyModules:SM0603-R-JRL, symbol R_US
- removed TP?: CONN_1, MyModules:TEST_POINT_LOOP_4592, symbol CONN_1
- removed U? (x2): TL072-, MyModules:TSSOP8-JRL, symbol TL072-
- added C? (x2): 100n, MyModules:SM0603-C-JRL, symbol C_US
- added C?: 33n, MyModules:SM0603-C-JRL, symbol C_US
- added C?: 1n, MyModules:SM0603-C-JRL, symbol C_US
- added C? (x2): 10μ, MyModules:SM0603-C-JRL, symbol C_US
- added J? (x2): JACK_MONO_SW, MyModules:PJ-301B-JACK-SLOTS, symbol JACK_MONO_SW
- added Q? (x4): MMBT3904, SOT-23, symbol MMBT3904
- added R? (x4): 100K, MyModules:SM0603-R-JRL, symbol R_US
- added R? (x2): 1.5meg, MyModules:SM0603-R-JRL, symbol R_US
- added R?: 2.2K, MyModules:SM0603-R-JRL, symbol R_US
- added R?: 150K, MyModules:SM0603-R-JRL, symbol R_US
- added R? (x2): 330K, MyModules:SM0603-R-JRL, symbol R_US
- added R?: 680K, MyModules:SM0603-R-JRL, symbol R_US
- added R?: 8.2K, MyModules:SM0603-R-JRL, symbol R_US
- added R? (x3): 10K, MyModules:SM0603-R-JRL, symbol R_US
- added R? (x2): 47K, MyModules:SM0603-R-JRL, symbol R_US
- added TP? (x3): CONN_1, MyModules:TEST_POINT_LOOP_4592, symbol CONN_1
- added U?: TL072-, MyModules:TSSOP8-JRL, symbol TL072-
- added VR?: 10K, MyModules:RV09AF-40-ALPHA-POT, symbol POT_US
- R?: value 33K -> 100K
Connections:
- net +12V: now also Q?.3 (C), Q?.3 (C), R?.1, R?.1
- net -12V: now also Q?.1 (B), R?.2, R?.2, R?.2
- net GND: now also U?.9 (In), C?.2, J?.1, J?.1, R?.1, R?.2, R?.2, R?.2, R?.2, R?.2, R?.2
- net LFO: now also TP?.1
- net PINK_NOISE: now also C?.1, J?.3, R?.1, TP?.1
- net WHITE_NOISE: now also C?.1, J?.3, R?.1, TP?.1
- net at U?.12 (Cd), U?.2 (Out), U?.4 (Cd): now also U?.12 (Cd), U?.4 (Cd)
- new net: C?.2, Q?.2 (E), R?.2
- new net: C?.1, R?.1, U?.5 (+)
- new net: R?.2, U?.6 (-)
- new net: C?.2, R?.1, R?.2, U?.7
- new net: C?.1, R?.1
- new net: Q?.1 (B), R?.1, R?.2
- new net: C?.1, Q?.1 (B), R?.1, R?.2 (x2)
- new net: Q?.2 (E), R?.1
- new net: C?.2, Q?.3 (C), R?.1, R?.2
- new net: R?.1, R?.1, VR?.2
- new net: R?.2, VR?.3
- new net: C?.2, Q?.2 (E), R?.1 (x2)
- now unconnected: U?.8 (Out)
- no-connect marks 12 -> 16
Other:
- note removed: "NEED TO ADD LEVEL\nADJUST TRIMMER HERE"
- note removed: "SEE HOW THIS WORKS IN\nVOICE SOCKET BOARD\nMAYBE JUST USE 100m 150/TR-808\nNOISE CIRCUIT HYBRID"
- note removed: "http://www.eeweb.com/blog/\nextreme_circuits/simple-white-noise-generator"
- moved on the sheet: U?D

Commit message: tidy up. next step: annotate
Parts:
- removed C? (x10): 100n, MyModules:SM0603-C-JRL, symbol C_US
- added C? (x3): 0.1µ, MyModules:SM0603-C-JRL, symbol C_US
- C?: value 100n -> 10n
Connections:
- net +12V: now also C?.1, C?.1, C?.2
- net GND: now also C?.1, C?.2, C?.2
Other:
- note added: "750 LFO S&H NOISE SLEW"
- note added: "DELAY\nTIME"
- note added: "FREQ"
- note added: "LEVEL\nTRIM"
- note added: "LFO"
- note added: "NOISE"
- note added: "NOISE \nLEVEL"
- note added: "POWER\n"
- note added: "RAMP\nADJUST"
- note added: "S&H CLOCK\nRATE"
- note added: "SAMPLE & HOLD"
- note added: "SLEW"
- note added: "SWITCHING LOGIC"
- note removed: "DECOUPLING"
- note removed: "LEVEL"
- note removed: "OP AMP DECOUPLING"
- note removed: "RAMP ADJUST"
- note removed: "S&H_RATE"
- moved on the sheet: C?, D?, J?, P?, Q?, Q?A, R?, SW?, TP?, U?, U?A, U?B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

Commit message: put PNP and NPN in LFO expo converter into single 3946 package, little bit of clean up
Parts:
- removed Q?: MMBT3904, SOT-23, symbol MMBT3904
- removed Q?: MMBT3906, SOT-23, symbol MMBT3906
- added J?: JACK_MONO_SW, MyModules:PJ-301B-JACK-SLOTS, symbol JACK_MONO_SW
- added Q? (x2): MBT3946DW, SOT-23, symbol MBT3946DW
- added R? (x2): 10, MyModules:SM0805-HAND, symbol R_US
- added R?: 1K, MyModules:SM0603-R-JRL, symbol R_US
- D?: value 1N914 -> 1N4148
- VR? (x2): footprint MyModules:RV09AF-40-ALPHA-POT -> MyModules:R_TRIM_3362P
- VR?: footprint MyModules:RV09AF-40-ALPHA-POT -> MyModules:RV16A-41-JRL
- gave numbers to parts that had none: 8
Connections:
- net +12V: now also U5.8 (V+), Q?.6 (C), R?.1; no longer P?.10 (P10), P?.9 (P9), U4.8 (V+)
- net -12V: now also U5.4 (V-), R?.1; no longer P?.1 (P1), P?.2 (P2), U4.4 (V-)
- net GND: now also J?.1, Q?.4 (E)
- net at C?.1, R?.1: now also U5.3 (+); no longer U5.5 (+)
- net at R?.2: now also U5.2 (-); no longer U5.6 (-)
- net at C?.2, R?.1, R?.2: now also U5.1; no longer U5.7
- net at R?.1, R?.2, VR?.2: now also Q?.2 (B)
- net at R?.1: now also Q?.1 (E), Q?.5 (B)
- net at R?.1: now also Q?.3 (C)
- net at R?.1, U1.5: now also U4.5 (+); no longer U4.3 (+)
- net S&H_OUT: no longer names the net of C?.2, R?.1, TP?.1, U?.7
- net S&H_OUT: now also R?.2
- new net: P?.1 (P1), P?.2 (P2), R?.2
- new net: P?.10 (P10), P?.9 (P9), R?.2
- new net: J?.3, R?.1
- new net: R?.1, U4.6 (-), U4.7
- no-connect marks 16 -> 17
Other:
- note added: "**"
- note added: "**Work out correct\ngain makeup here"
- note added: "Ian Fritz Super Sampe & Hold\nhttp://ijfritz.byethost4.com/super_sh_rand_web.pdf"
- note added: "PINK OR WHITE NOISE \nFOR S&H INPUT?"
- note added: "S&H EXT CLK"
- note added: "S&H OUT"
- note added: "Yusynth S&H sample\ngate generator"
- note removed: "B"
- note removed: "Ian Fritz Super Sampe & Hold"
- note removed: "S&H_EXT_CLK"

Commit message: added filtered rails for noise circuit a la TR-808
Parts:
- added C? (x2): 10μF, MyModules:2MM-POL-CAP, symbol CP_US
- added R? (x2): 100, MyModules:SM0603-R-JRL, symbol R_US
- VR? (x3): footprint MyModules:RV09AF-40-ALPHA-POT -> MyModules:RV16A-41-JRL
- VR? (x2): footprint MyModules:RV09AF-40-ALPHA-POT -> MyModules:Bourns_3362P
- gave numbers to parts that had none: 5
Connections:
- net +12V: now also R?.2; no longer Q?.3 (C), Q?.3 (C), R?.1, R?.1, U5.8 (V+)
- net -12V: now also R?.2; no longer Q?.1 (B), R?.2, R?.2, R?.2
- net GND: now also C?.1 (+), C?.2 (-)
- net at Q3.1 (S): now also Q3.4 (S); no longer Q3.1 (S)
- net at D?.1 (A), Q3.2 (G), U10.1: now also Q3.5 (G); no longer Q3.2 (G)
- net at Q4.6 (D), R?.1: now also Q3.3 (D); no longer Q3.6 (D)
- net at Q4.1 (S): now also Q4.4 (S); no longer Q4.1 (S)
- net at D?.2 (K), Q4.2 (G), R?.2: now also Q4.5 (G); no longer Q4.2 (G)
- net at C?.1, U?.2 (-): now also Q4.3 (D); no longer Q4.6 (D)
- new net +Vn: C?.1 (+), Q?.3 (C), Q?.3 (C), R?.1, R?.1, R?.1, U5.8 (V+)
- new net -Vn: C?.2 (-), Q?.1 (B), R?.1, R?.2, R?.2, R?.2
Other:
- note added: "FREQ\nTRIM"
- note added: "NOISE CIRCUIT\nPOWER FILTERING"
- moved on the sheet: C?, J?, Q?, R?, TP?, U5A, VR?

Commit message: annotated, footprints assinged, netlist generated
Parts:
- gave numbers to parts that had none: 224
Connections:
- net +12V: now also U1.11 (V+)
- net -12V: now also U1.6 (V-)
- net at R58.1, U4.5 (+): now also U1.12; no longer U1.5
- net at R48.2: now also U1.16; no longer U1.1
- net at R45.1, R46.1: now also U1.14 (+); no longer U1.3 (+)
- net at R47.1: now also U1.13 (-); no longer U1.4 (-)
- no-connect marks 17 -> 19
Other:
- moved on the sheet: C1, C10, C2, C21, C22, C3, C30, C31, C34, C35, C36, C37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
