File: 750 LFO S&H NOISE SLEW.sch (KiCad schematic (older format))
At the start: 237 parts, among them J1 JACK_MONO_SW, J10 JACK_MONO_SW, J11 JACK_MONO_SW, J2 JACK_MONO_SW, J3 JACK_MONO_SW, J4 JACK_MONO_SW, J5 JACK_MONO_SW, J6 JACK_MONO_SW, J7 JACK_MONO_SW, J8 JACK_MONO_SW, J9 JACK_MONO_SW, P1 CONN_02X01, P2 CONN_02X01, P3 CONN_02X05, Q1 MMBT3904, Q10 MMBT3904, Q11 J112, Q12 MMBT3906, Q13 J112, Q14 J112, Q15 MMBT3904, Q16 MMBT3904, Q2 MMBT3904, Q3 2N7002, Q4 2N7002, Q5 MBT3946DW, Q6 DMMT3904W, Q7 MMBT3904, Q8 MMBT3904, Q9 MMBT3904, SW1 KS-01Q, SW2 KS-01Q, U1 LM13700, U10 TL072-, U11 TL072-, U12 MAX9945, U13 DG409, U14 DG409, U2 TL072-, U3 TL072-, U4 TL072-, U5 TL072-, U6 CD40106, U7 CD4027, U8 CD4027, U9 TL072-

Commit message: started placing comps on PCB. jacks, pots and LEDs placed
Parts:
- C27: footprint (none) -> MyModules:2MM-POL-CAP
- C34: footprint MyModules:CAP-5MM-BOX-0805-COMBO -> MyModules:2MM-POL-CAP
- P1, P2: footprint (none) -> Pin_Headers:Pin_Header_Straight_1x02
- Q1, Q10, Q12, Q2, Q7, Q8, Q9: footprint SOT-23 -> MyModules:SOT23-132-JRL
- Q5: footprint SOT-23 -> MyModules:SOT363-JRL
- U13, U14: footprint (none) -> MyModules:SO16-JRL
Changed lines of the file:
@@
 F 0 "C34" H 11275 4575 50  0000 L CNN
 F 1 "4.7μ" H 11275 4375 50  0000 L CNN
-F 2 "MyModules:CAP-5MM-BOX-0805-COMBO" H 11225 4475 60  0001 C CNN
+F 2 "MyModules:2MM-POL-CAP" H 11225 4475 60  0001 C CNN
 F 3 "" H 11225 4475 60  0000 C CNN
 	1    11225 4475
@@
 F 0 "U13" H 18275 8500 60  0000 C CNN
 F 1 "DG409" H 18875 8500 60  0000 C CNN
-F 2 "" H 18625 7800 60  0000 C CNN
+F 2 "MyModules:SO16-JRL" H 18625 7800 60  0001 C CNN
 F 3 "" H 18625 7800 60  0000 C CNN
 	1    18625 7800
@@
 F 0 "U14" H 18275 11875 60  0000 C CNN
 F 1 "DG409" H 18875 11875 60  0000 C CNN
-F 2 "" H 18625 11175 60  0000 C CNN
+F 2 "MyModules:SO16-JRL" H 18625 11175 60  0001 C CNN
 F 3 "" H 18625 11175 60  0000 C CNN
 	1    18625 11175
@@
 F 0 "Q10" H 6225 11000 50  0000 L CNN
 F 1 "MMBT3904" H 6225 10925 50  0000 L CNN
-F 2 "SOT-23" H 6225 10850 50  0001 L CIN
+F 2 "MyModules:SOT23-132-JRL" H 6225 10850 50  0001 L CIN
 F 3 "" H 6025 10925 50  0000 L CNN
 	1    6025 10925
@@
 F 0 "P1" V 2225 11375 50  0000 C CNN
 F 1 "CONN_02X01" V 2150 11175 50  0000 C CNN
-F 2 "" H 2350 10300 60  0000 C CNN
+F 2 "Pin_Headers:Pin_Header_Straight_1x02" H 2350 10300 60  0001 C CNN
 F 3 "" H 2350 10300 60  0000 C CNN
 	1    2350 11500
@@
 F 0 "P2" H 3900 12925 50  0000 C CNN
 F 1 "CONN_02X01" H 3800 12725 50  0000 C CNN
-F 2 "" H 3775 11625 60  0000 C CNN
+F 2 "Pin_Headers:Pin_Header_Straight_1x02" H 3775 11625 60  0001 C CNN
 F 3 "" H 3775 11625 60  0000 C CNN
 	1    3775 12825
@@
 F 0 "Q8" H 5425 13050 50  0000 L CNN
 F 1 "MMBT3904" H 5075 12950 50  0000 L CNN
-F 2 "SOT-23" H 5700 12750 50  0001 L CIN
+F 2 "MyModules:SOT23-132-JRL" H 5700 12750 50  0001 L CIN
 F 3 "" H 5500 12825 50  0000 L CNN
 	1    5500 12825
@@
 F 0 "C27" H 6125 12800 50  0000 L CNN
 F 1 "4.7μ" H 6125 12600 50  0000 L CNN
-F 2 "" H 6075 12700 60  0000 C CNN
+F 2 "MyModules:2MM-POL-CAP" H 6075 12700 60  0001 C CNN
 F 3 "" H 6075 12700 60  0000 C CNN
 	1    6075 12700
@@
 F 0 "Q12" V 8025 14050 50  0000 L CNN
 F 1 "MMBT3906" V 7950 14050 50  0000 L CNN
-F 2 "SOT-23" H 7925 13950 50  0001 L CIN
+F 2 "MyModules:SOT23-132-JRL" H 7925 13950 50  0001 L CIN
 F 3 "" H 7725 14025 50  0000 L CNN
 	1    7725 14025
@@
 F 0 "Q1" V 1800 4050 50  0000 L CNN
 F 1 "MMBT3904" V 1725 3750 50  0000 L CNN
-F 2 "SOT-23" H 2025 3500 50  0001 L CIN
+F 2 "MyModules:SOT23-132-JRL" H 2025 3500 50  0001 L CIN
 F 3 "" H 1825 3575 50  0000 L CNN
 	1    1825 3575
@@
 F 0 "Q2" H 2925 3400 50  0000 L CNN
 F 1 "MMBT3904" H 2925 3325 50  0000 L CNN
-F 2 "SOT-23" H 2925 3400 50  0001 L CIN
+F 2 "MyModules:SOT23-132-JRL" H 2925 3400 50  0001 L CIN
 F 3 "" H 2725 3475 50  0000 L CNN
 	1    2725 3475
@@
 F 0 "Q9" H 5975 3000 50  0000 L CNN
 F 1 "MMBT3904" H 5975 2925 50  0000 L CNN
-F 2 "SOT-23" H 6000 2775 50  0001 L CIN
+F 2 "MyModules:SOT23-132-JRL" H 6000 2775 50  0001 L CIN
 F 3 "" H 5800 2850 50  0000 L CNN
 	1    5800 2850
@@
 F 0 "Q7" H 5475 4375 50  0000 L CNN
 F 1 "MMBT3904" H 5475 4300 50  0000 L CNN
-F 2 "SOT-23" H 5500 4150 50  0001 L CIN
+F 2 "MyModules:SOT23-132-JRL" H 5500 4150 50  0001 L CIN
 F 3 "" H 5300 4225 50  0000 L CNN
 	1    5300 4225
@@
 F 0 "Q5" H 4925 7775 50  0000 L CNN
 F 1 "MBT3946DW" H 4925 7700 50  0000 L CNN
-F 2 "SOT-23" H 4925 7625 50  0001 L CIN
+F 2 "MyModules:SOT363-JRL" H 4925 7625 50  0001 L CIN
 F 3 "" H 4725 7700 50  0000 L CNN
 	1    4725 7700
@@
 F 0 "Q5" H 5425 8200 50  0000 L CNN
 F 1 "MBT3946DW" H 5425 8125 50  0000 L CNN
-F 2 "SOT-23" H 5425 8050 50  0001 L CIN
+F 2 "MyModules:SOT363-JRL" H 5425 8050 50  0001 L CIN
 F 3 "" H 5225 8125 50  0000 L CNN
 	2    5225 8125

Commit message: more component placement
Parts:
- C30, C31: footprint MyModules:SM0603-C-JRL -> MyModules:SM0805-HAND
- C43: value 0.47μ -> 1μ
Connections:
- net +12V: now also U5.8 (V+)
- net +Vn: no longer U5.8 (V+)
Changed lines of the file:
@@
 P 25300 10750
 F 0 "C43" H 25350 10850 50  0000 L CNN
-F 1 "0.47μ" H 25350 10650 50  0000 L CNN
+F 1 "1μ" H 25350 10650 50  0000 L CNN
 F 2 "MyModules:SM0603-C-JRL" H 25300 10750 60  0001 C CNN
 F 3 "" H 25300 10750 60  0000 C CNN
@@
 F 0 "C31" V 6675 3025 50  0000 L CNN
 F 1 "10μ" V 6350 3000 50  0000 L CNN
-F 2 "MyModules:SM0603-C-JRL" H 6500 3075 60  0001 C CNN
+F 2 "MyModules:SM0805-HAND" H 6500 3075 60  0001 C CNN
 F 3 "" H 6500 3075 60  0000 C CNN
 	1    6500 3075
@@
 F 0 "C30" V 6650 4400 50  0000 L CNN
 F 1 "10μ" V 6325 4375 50  0000 L CNN
-F 2 "MyModules:SM0603-C-JRL" H 6475 4450 60  0001 C CNN
+F 2 "MyModules:SM0805-HAND" H 6475 4450 60  0001 C CNN
 F 3 "" H 6475 4450 60  0000 C CNN
 	1    6475 4450
@@
 Text Notes 29375 20675 0    200  ~ 40
 750 LFO S&H NOISE SLEW
-$Comp
-L -12V #PWR0147
-U 1 1 56FD9029
-P 3850 3250
-F 0 "#PWR0147" H 3850 3350 30  0001 C CNN
-F 1 "-12V" H 3850 3425 50  0000 C CNN
-F 2 "~" H 3850 3250 60  0000 C CNN
-F 3 "~" H 3850 3250 60  0000 C CNN
-	1    3850 3250
-	-1   0    0    1
-$EndComp
 Text Notes 17050 7175 0    60   ~ 0
 PINK OR WHITE NOISE \nFOR S&H INPUT?
@@
 NoConn ~ 20525 4225
 $Comp
-L GND_E #PWR0148
+L GND_E #PWR0147
 U 1 1 57033524
 P 20525 4575
-F 0 "#PWR0148" V 20525 4575 30  0001 C CNN
+F 0 "#PWR0147" V 20525 4575 30  0001 C CNN
 F 1 "GND_E" H 20525 4505 30  0001 C CNN
 F 2 "" H 20525 4575 60  0000 C CNN
@@
 FREQ\nTRIM
 $Comp
-L +Vn #PWR0149
+L +Vn #PWR0148
 U 1 1 56EF2608
 P 5900 2575
-F 0 "#PWR0149" H 5900 2425 50  0001 C CNN
+F 0 "#PWR0148" H 5900 2425 50  0001 C CNN
 F 1 "+Vn" H 5875 2725 50  0000 C CNN
 F 2 "" H 5900 2575 60  0000 C CNN
@@
 $EndComp
 $Comp
-L -Vn #PWR0150
+L -Vn #PWR0149
 U 1 1 56EFA2A2
 P 5400 4875
-F 0 "#PWR0150" H 5400 4985 50  0001 C CNN
+F 0 "#PWR0149" H 5400 4985 50  0001 C CNN
 F 1 "-Vn" H 5380 4715 50  0000 C CNN
 F 2 "" H 5400 4875 60  0000 C CNN
@@
 $Comp
 L +Vn #PWR0151
-U 1 1 56EFC686
-P 3850 2450
-F 0 "#PWR0151" H 3850 2300 50  0001 C CNN
-F 1 "+Vn" H 3825 2600 50  0000 C CNN
-F 2 "" H 3850 2450 60  0000 C CNN
-F 3 "" H 3850 2450 60  0000 C CNN
-	1    3850 2450
-	1    0    0    -1
-$EndComp
-$Comp
-L +Vn #PWR0152
 U 1 1 56EFDE3E
 P 2825 2500
-F 0 "#PWR0152" H 2825 2350 50  0001 C CNN
+F 0 "#PWR0151" H 2825 2350 50  0001 C CNN
 F 1 "+Vn" H 2800 2650 50  0000 C CNN
 F 2 "" H 2825 2500 60  0000 C CNN
@@
 $EndComp
 $Comp
-L +Vn #PWR0153
+L +Vn #PWR0152
 U 1 1 56EFF4FD
 P 2050 2975
-F 0 "#PWR0153" H 2050 2825 50  0001 C CNN
+F 0 "#PWR0152" H 2050 2825 50  0001 C CNN
 F 1 "+Vn" H 2025 3125 50  0000 C CNN
 F 2 "" H 2050 2975 60  0000 C CNN
@@
 $EndComp
 $Comp
-L +Vn #PWR0154
+L +Vn #PWR0153
 U 1 1 56F0225A
 P 5400 3950
-F 0 "#PWR0154" H 5400 3800 50  0001 C CNN
+F 0 "#PWR0153" H 5400 3800 50  0001 C CNN
 F 1 "+Vn" H 5375 4100 50  0000 C CNN
 F 2 "" H 5400 3950 60  0000 C CNN
@@
 $EndComp
 $Comp
-L -Vn #PWR0155
+L -Vn #PWR0154
 U 1 1 56F042F9
 P 2825 4075
-F 0 "#PWR0155" H 2825 4185 50  0001 C CNN
+F 0 "#PWR0154" H 2825 4185 50  0001 C CNN
 F 1 "-Vn" H 2805 3915 50  0000 C CNN
 F 2 "" H 2825 4075 60  0000 C CNN
@@
 $EndComp
 $Comp
-L -Vn #PWR0156
+L -Vn #PWR0155
 U 1 1 56F05CAD
 P 2500 4075
-F 0 "#PWR0156" H 2500 4185 50  0001 C CNN
+F 0 "#PWR0155" H 2500 4185 50  0001 C CNN
 F 1 "-Vn" H 2480 3915 50  0000 C CNN
 F 2 "" H 2500 4075 60  0000 C CNN
@@
 $EndComp
 $Comp
-L -Vn #PWR0157
+L -Vn #PWR0156
 U 1 1 56F05FAC
 P 1825 4075
-F 0 "#PWR0157" H 1825 4185 50  0001 C CNN
+F 0 "#PWR0156" H 1825 4185 50  0001 C CNN
 F 1 "-Vn" H 1805 3915 50  0000 C CNN
 F 2 "" H 1825 4075 60  0000 C CNN
@@
 $EndComp
 $Comp
-L GND_E #PWR0158
+L GND_E #PWR0157
 U 1 1 56F0AF31
 P 1100 5225
-F 0 "#PWR0158" V 1100 5225 30  0001 C CNN
+F 0 "#PWR0157" V 1100 5225 30  0001 C CNN
 F 1 "GND_E" H 1100 5155 30  0001 C CNN
 F 2 "" H 1100 5225 60  0000 C CNN
@@
 $EndComp
 $Comp
-L +12V #PWR0159
+L +12V #PWR0158
 U 1 1 56F0AF37
 P 2100 4450
-F 0 "#PWR0159" H 2100 4300 50  0001 C CNN
+F 0 "#PWR0158" H 2100 4300 50  0001 C CNN
 F 1 "+12V" H 2100 4590 50  0000 C CNN
 F 2 "" H 2100 4450 60  0000 C CNN
@@
 $EndComp
 $Comp
-L -12V #PWR0160
+L -12V #PWR0159
 U 1 1 56F0AF49
 P 2125 5550
-F 0 "#PWR0160" H 2125 5400 50  0001 C CNN
+F 0 "#PWR0159" H 2125 5400 50  0001 C CNN
 F 1 "-12V" H 2125 5690 50  0000 C CNN
 F 2 "" H 2125 5550 60  0000 C CNN
@@
 	1525 5450 1625 5450
 $Comp
-L +Vn #PWR0161
+L +Vn #PWR0160
 U 1 1 56F14B5B
 P 1525 4450
-F 0 "#PWR0161" H 1525 4300 50  0001 C CNN
+F 0 "#PWR0160" H 1525 4300 50  0001 C CNN
 F 1 "+Vn" H 1500 4600 50  0000 C CNN
 F 2 "" H 1525 4450 60  0000 C CNN
@@
 	1525 4450 1525 4550
 $Comp
-L -Vn #PWR0162
+L -Vn #PWR0161
 U 1 1 56F16240
 P 1525 5550
-F 0 "#PWR0162" H 1525 5660 50  0001 C CNN
+F 0 "#PWR0161" H 1525 5660 50  0001 C CNN
 F 1 "-Vn" H 1505 5390 50  0000 C CNN
 F 2 "" H 1525 5550 60  0000 C CNN
@@
 NOISE CIRCUIT\nPOWER FILTERING
 $Comp
-L -12V #PWR0163
+L -12V #PWR0162
 U 1 1 56F5C56C
 P 8775 15350
-F 0 "#PWR0163" H 8775 15450 30  0001 C CNN
+F 0 "#PWR0162" H 8775 15450 30  0001 C CNN
 F 1 "-12V" H 8775 15525 50  0000 C CNN
 F 2 "~" H 8775 15350 60  0000 C CNN
@@
 $EndComp
 $Comp
-L +12V #PWR0164
+L +12V #PWR0163
 U 1 1 56F5DE77
 P 8775 14550
-F 0 "#PWR0164" H 8775 14400 50  0001 C CNN
+F 0 "#PWR0163" H 8775 14400 50  0001 C CNN
 F 1 "+12V" H 8775 14690 50  0000 C CNN
 F 2 "" H 8775 14550 60  0000 C CNN
@@
 NoConn ~ 7275 8150
 NoConn ~ 8575 14950
+$Comp
+L +12V #PWR?
+U 1 1 56FB3627
+P 3850 2450
+F 0 "#PWR?" H 3850 2300 50  0001 C CNN
+F 1 "+12V" H 3850 2590 50  0000 C CNN
+F 2 "" H 3850 2450 60  0000 C CNN
+F 3 "" H 3850 2450 60  0000 C CNN
+	1    3850 2450
+	-1   0    0    -1
+$EndComp
+$Comp
+L -12V #PWR?
+U 1 1 56FB6932
+P 3850 3250
+F 0 "#PWR?" H 3850 3350 30  0001 C CNN
+F 1 "-12V" H 3850 3425 60  0000 C CNN
+F 2 "~" H 3850 3250 60  0000 C CNN
+F 3 "~" H 3850 3250 60  0000 C CNN
+	1    3850 3250
+	-1   0    0    1
+$EndComp
 $EndSCHEMATC

Commit message: placing components, starting a bit from scratch
Parts:
- C44: footprint MyModules:SM0805-HAND -> MyModules:CAP-5MM-BOX-0805-COMBO
Other:
- note added: "SHORT R109 to prevent \nvoltage drop with >1 \noutputs connected?"
Changed lines of the file:
@@
 F 0 "C44" H 25950 3575 50  0000 L CNN
 F 1 "470n" H 25950 3375 50  0000 L CNN
-F 2 "MyModules:SM0805-HAND" H 25900 3475 60  0001 C CNN
+F 2 "MyModules:CAP-5MM-BOX-0805-COMBO" H 25900 3475 60  0001 C CNN
 F 3 "~" H 25900 3475 60  0000 C CNN
 	1    25900 3475
@@
 $EndComp
 $Comp
-L +Vn #PWR0151
+L +Vn #PWR0150
 U 1 1 56EFDE3E
 P 2825 2500
-F 0 "#PWR0151" H 2825 2350 50  0001 C CNN
+F 0 "#PWR0150" H 2825 2350 50  0001 C CNN
 F 1 "+Vn" H 2800 2650 50  0000 C CNN
 F 2 "" H 2825 2500 60  0000 C CNN
@@
 $EndComp
 $Comp
-L +Vn #PWR0152
+L +Vn #PWR0151
 U 1 1 56EFF4FD
 P 2050 2975
-F 0 "#PWR0152" H 2050 2825 50  0001 C CNN
+F 0 "#PWR0151" H 2050 2825 50  0001 C CNN
 F 1 "+Vn" H 2025 3125 50  0000 C CNN
 F 2 "" H 2050 2975 60  0000 C CNN
@@
 $EndComp
 $Comp
-L +Vn #PWR0153
+L +Vn #PWR0152
 U 1 1 56F0225A
 P 5400 3950
-F 0 "#PWR0153" H 5400 3800 50  0001 C CNN
+F 0 "#PWR0152" H 5400 3800 50  0001 C CNN
 F 1 "+Vn" H 5375 4100 50  0000 C CNN
 F 2 "" H 5400 3950 60  0000 C CNN
@@
 $EndComp
 $Comp
-L -Vn #PWR0154
+L -Vn #PWR0153
 U 1 1 56F042F9
 P 2825 4075
-F 0 "#PWR0154" H 2825 4185 50  0001 C CNN
+F 0 "#PWR0153" H 2825 4185 50  0001 C CNN
 F 1 "-Vn" H 2805 3915 50  0000 C CNN
 F 2 "" H 2825 4075 60  0000 C CNN
@@
 $EndComp
 $Comp
-L -Vn #PWR0155
+L -Vn #PWR0154
 U 1 1 56F05CAD
 P 2500 4075
-F 0 "#PWR0155" H 2500 4185 50  0001 C CNN
+F 0 "#PWR0154" H 2500 4185 50  0001 C CNN
 F 1 "-Vn" H 2480 3915 50  0000 C CNN
 F 2 "" H 2500 4075 60  0000 C CNN
@@
 $EndComp
 $Comp
-L -Vn #PWR0156
+L -Vn #PWR0155
 U 1 1 56F05FAC
 P 1825 4075
-F 0 "#PWR0156" H 1825 4185 50  0001 C CNN
+F 0 "#PWR0155" H 1825 4185 50  0001 C CNN
 F 1 "-Vn" H 1805 3915 50  0000 C CNN
 F 2 "" H 1825 4075 60  0000 C CNN
@@
 $EndComp
 $Comp
-L GND_E #PWR0157
+L GND_E #PWR0156
 U 1 1 56F0AF31
 P 1100 5225
-F 0 "#PWR0157" V 1100 5225 30  0001 C CNN
+F 0 "#PWR0156" V 1100 5225 30  0001 C CNN
 F 1 "GND_E" H 1100 5155 30  0001 C CNN
 F 2 "" H 1100 5225 60  0000 C CNN
@@
 $EndComp
 $Comp
-L +12V #PWR0158
+L +12V #PWR0157
 U 1 1 56F0AF37
 P 2100 4450
-F 0 "#PWR0158" H 2100 4300 50  0001 C CNN
+F 0 "#PWR0157" H 2100 4300 50  0001 C CNN
 F 1 "+12V" H 2100 4590 50  0000 C CNN
 F 2 "" H 2100 4450 60  0000 C CNN
@@
 $EndComp
 $Comp
-L -12V #PWR0159
+L -12V #PWR0158
 U 1 1 56F0AF49
 P 2125 5550
-F 0 "#PWR0159" H 2125 5400 50  0001 C CNN
+F 0 "#PWR0158" H 2125 5400 50  0001 C CNN
 F 1 "-12V" H 2125 5690 50  0000 C CNN
 F 2 "" H 2125 5550 60  0000 C CNN
@@
 	1525 5450 1625 5450
 $Comp
-L +Vn #PWR0160
+L +Vn #PWR0159
 U 1 1 56F14B5B
 P 1525 4450
-F 0 "#PWR0160" H 1525 4300 50  0001 C CNN
+F 0 "#PWR0159" H 1525 4300 50  0001 C CNN
 F 1 "+Vn" H 1500 4600 50  0000 C CNN
 F 2 "" H 1525 4450 60  0000 C CNN
@@
 	1525 4450 1525 4550
 $Comp
-L -Vn #PWR0161
+L -Vn #PWR0160
 U 1 1 56F16240
 P 1525 5550
-F 0 "#PWR0161" H 1525 5660 50  0001 C CNN
+F 0 "#PWR0160" H 1525 5660 50  0001 C CNN
 F 1 "-Vn" H 1505 5390 50  0000 C CNN
 F 2 "" H 1525 5550 60  0000 C CNN
@@
 NOISE CIRCUIT\nPOWER FILTERING
 $Comp
-L -12V #PWR0162
+L -12V #PWR0161
 U 1 1 56F5C56C
 P 8775 15350
-F 0 "#PWR0162" H 8775 15450 30  0001 C CNN
+F 0 "#PWR0161" H 8775 15450 30  0001 C CNN
 F 1 "-12V" H 8775 15525 50  0000 C CNN
 F 2 "~" H 8775 15350 60  0000 C CNN
@@
 $EndComp
 $Comp
-L +12V #PWR0163
+L +12V #PWR0162
 U 1 1 56F5DE77
 P 8775 14550
-F 0 "#PWR0163" H 8775 14400 50  0001 C CNN
+F 0 "#PWR0162" H 8775 14400 50  0001 C CNN
 F 1 "+12V" H 8775 14690 50  0000 C CNN
 F 2 "" H 8775 14550 60  0000 C CNN
@@
 NoConn ~ 8575 14950
 $Comp
-L +12V #PWR?
+L +12V #PWR0163
 U 1 1 56FB3627
 P 3850 2450
-F 0 "#PWR?" H 3850 2300 50  0001 C CNN
+F 0 "#PWR0163" H 3850 2300 50  0001 C CNN
 F 1 "+12V" H 3850 2590 50  0000 C CNN
 F 2 "" H 3850 2450 60  0000 C CNN
@@
 $EndComp
 $Comp
-L -12V #PWR?
+L -12V #PWR0164
 U 1 1 56FB6932
 P 3850 3250
-F 0 "#PWR?" H 3850 3350 30  0001 C CNN
+F 0 "#PWR0164" H 3850 3350 30  0001 C CNN
 F 1 "-12V" H 3850 3425 60  0000 C CNN
 F 2 "~" H 3850 3250 60  0000 C CNN
@@
 	-1   0    0    1
 $EndComp
+Text Notes 27100 4025 0    50   ~ 0
+SHORT R109 to prevent \nvoltage drop with >1 \noutputs connected?
+Wire Notes Line
+	27850 3250 27850 3775
 $EndSCHEMATC
