File: 750 LFO S&H NOISE SLEW.sch (KiCad schematic (older format))
At the start: 232 parts, among them J1 PJ301BM, J10 PJ301BM, J11 PJ301BM, J2 PJ301BM, J3 PJ301BM, J4 PJ301BM, J5 JACK_MONO_SW, J6 PJ301BM, J7 JACK_MONO_SW, J8 PJ301BM, J9 PJ301BM, P1 CONN_01X03, P3 CONN_02X05, Q1 MMBT3904, Q10 MMBT3904, Q11 J112, Q12 MMBT3906, Q13 J112, Q14 J112, Q15 MMBT3904, Q16 MMBT3904, Q2 MMBT3904, Q3 2N7002, Q4 2N7002, Q5 MBT3946DW, Q6 MBT3946DW, Q7 MMBT3904, Q8 MMBT3904, Q9 MMBT3904, SW1 KS-01Q, SW2 KS-01Q, SW3 SPDT, U1 LM13700, U10 TL072-, U11 TL072-, U12 MAX9945, U13 DG409, U14 DG409, U15 TS321, U2 TL072-, U3 TL072-, U4 TL072-, U5 TL072-, U6 CD40106, U7 CD4027, U8 CD4027, U9 TL072-

Commit message: silkscreen tweaked, ready for panel check
Other:
- note added: "Use C945 here"

Commit message: working on v1.3. almost done
Parts:
- added C1: 0.1µ, MyModules:SM0603-C-JRL, symbol C_US
- R96, R97: value 2.2K -> 3.3K
- VR9: value 5K -> 10K
Connections:
- net +12V: now also C1.1
- net GND: now also C1.2
Other:
- note added: "850 LFO S&H NOISE SLEW"
- note added: "Changed C27 to\nNP ceramic"
- note added: "Increase to 6.8\nor 10 to extend\ndelay time?"
- note added: "NOISE AMPLIFIER CONFIGURED\nFOR BJT 4558. USE 4558 OR RE-\nCONFIGURE FOR TL07X?"
- note removed: "750 LFO S&H NOISE SLEW"
- note removed: "Change C27 to\nNP ceramic"
- note removed: "Yusynth S&H sample\ngate generator"

Commit message: added a couple of superflurous output protection resistors
Parts:
- added R110, R111: 1K, MyModules:SM0603-R-JRL, symbol R_US
Connections:
- net S&H_INT_CLK: now also R110.1; no longer R56.1, U9.1, VR6.3
- net at C37.2, R98.1, R99.2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: no longer P1.1 (P1)
- net at C34.2, R55.1, U9.7: now also R111.2; no longer J11.3
- net at J8.3, R99.1: now also P1.1 (P1)
- new net: R110.2, R56.1, U9.1, VR6.3
- new net: J11.3, R111.1
Other:
- note added: "current limit R\nhere?"
- note added: "current limit\nR here?"
- note removed: "add TL072 to handle S&H buffering\nand also bias and scale S&H clock to SLEW?"

Commit message: changed R25 value to improve LFO reset response
Parts:
- R25: value 10K -> 22K
Other:
- note added: "Adjust R25 to 22K\nfor reliable retriggering\nwith 5V gate"
Changed lines of the file:
@@
 P 5100 9600
 F 0 "R25" H 5225 9650 50  0000 C CNN
-F 1 "10K" H 5275 9575 50  0000 C CNN
+F 1 "22K" H 5275 9575 50  0000 C CNN
 F 2 "MyModules:SM0603-R-JRL" H 5100 9600 60  0001 C CNN
 F 3 "" H 5100 9600 60  0000 C CNN
@@
 	21425 3850 20625 3850
 Connection ~ 20625 3850
+Text Notes 3925 9450 0    60   ~ 0
+Adjust R25 to 22K\nfor reliable retriggering\nwith 5V gate
 $EndSCHEMATC

Commit message: notes
Parts:
- R1: value 270K -> 220K
- R72: value 330K -> 150K
- R8: value 150K -> 120K
Other:
- note added: "Changed R8 to 120K\nGives 100 mHz as\nlowest LFO rate"
- note added: "LOG"
- note added: "Reduce R72 to 150K\nto get 10Vpp TRI \noutput"
- note removed: "BIAS down further\nfor lower min freq?"
- note removed: "LIN or LOG?\nI think LIN"
Changed lines of the file:
@@
 P 2525 8050
 F 0 "R8" H 2650 8100 50  0000 C CNN
-F 1 "150K" H 2700 8025 50  0000 C CNN
+F 1 "120K" H 2700 8025 50  0000 C CNN
 F 2 "MyModules:SM0603-R-JRL" H 2525 8050 60  0001 C CNN
 F 3 "" H 2525 8050 60  0000 C CNN
@@
 P 11900 6950
 F 0 "R72" V 11980 6950 50  0000 C CNN
-F 1 "330K" V 11820 6950 50  0000 C CNN
+F 1 "150K" V 11820 6950 50  0000 C CNN
 F 2 "MyModules:SM0603-R-JRL" H 11900 6950 60  0001 C CNN
 F 3 "" H 11900 6950 60  0000 C CNN
@@
 Wire Wire Line
 	19150 4025 19150 4275
-Text Notes 2025 8650 0    60   ~ 0
-BIAS down further\nfor lower min freq?
+Text Notes 2100 8750 0    60   ~ 0
+Changed R8 to 120K\nGives 100 mHz as\nlowest LFO rate
 Text Notes 12500 4375 0    50   ~ 0
 S&H TRI OUT
@@
 P 3375 6550
 F 0 "R1" V 3455 6550 50  0000 C CNN
-F 1 "270K" V 3295 6550 50  0000 C CNN
+F 1 "220K" V 3295 6550 50  0000 C CNN
 F 2 "MyModules:SM0603-R-JRL" H 3375 6550 60  0001 C CNN
 F 3 "" H 3375 6550 60  0000 C CNN
@@
 RANGE
 Text Notes 5275 11900 0    60   ~ 0
-LIN or LOG?\nI think LIN
+LOG
 Wire Wire Line
 	6825 2700 6825 3175
@@
 Text Notes 3925 9450 0    60   ~ 0
 Adjust R25 to 22K\nfor reliable retriggering\nwith 5V gate
+Text Notes 11550 6800 0    60   ~ 0
+Reduce R72 to 150K\nto get 10Vpp TRI \noutput
 $EndSCHEMATC

Commit message: LFO voltage reference added and routed"
l
q
;ksadjf

q
exit
"
Parts:
- removed R41: 10, MyModules:SM0805-HAND, symbol R_US
- added C2: 1000p, MyModules:SM0603-C-JRL, symbol C_US
- added D24: LM4040-10, MyModules:SOT23-132-JRL, symbol LM4040
- added F1, F2: PTC 0.1A, Capacitors_SMD:C_0805, symbol FUSE
- D3, D4: value D -> S1BB
- R1: value 220K -> 180K
- R40: value 10 -> 1K; footprint MyModules:SM0805-HAND -> MyModules:SM0603-R-JRL
Connections:
- net +12V: now also F1.2; no longer C1.1, Q5.6 (C), R1.2, VR1.3, VR3.3
- net -12V: now also F2.2
- net GND: now also C2.2, D24.2 (A)
- net at Q15.1 (B), R78.2: now also C2.1
- net at P3.1 (P1), P3.2 (P2): now also F2.1
- net at P3.10 (P10), P3.9 (P9): now also F1.1; no longer R40.2
- new net +10V: C1.1, D24.1 (K), Q5.6 (C), R1.2, R40.2, VR1.3, VR3.3
- no-connect marks 19 -> 20
Other:
- note removed: "PINK OR WHITE NOISE \nFOR S&H INPUT?"
- moved on the sheet: C1, R78, R80

Commit message: tweakings
Other:
- note added: "SYSTEM80 INC. 2017"
Changed lines of the file:
@@
 	12725 2275 12500 2275
 Connection ~ 12500 2275
+Text Notes 29400 20050 0    200  ~ 40
+SYSTEM80 INC. 2017
 $EndSCHEMATC

Commit message: 850 gerbers plotted
Parts:
- C2: value 1000p -> 1n
Other:
- note added: "'850' modulation/noise source"
- note added: "1.4"
- note added: "Changed R8 to 120K\nGives 50 mHz as\nlowest LFO rate"
- note added: "LFO, S&H, NOISE, SLEW EURORACK MODULE"
- note removed: "850 LFO S&H NOISE SLEW"
- note removed: "Changed R8 to 120K\nGives 100 mHz as\nlowest LFO rate"
Changed lines of the file:
@@
 Wire Notes Line
 	6825 13975 6550 13975
-Text Notes 29375 20675 0    200  ~ 40
-850 LFO S&H NOISE SLEW
 $Comp
 L MBT3946DW Q5
@@
 	19150 4025 19150 4275
 Text Notes 2100 8750 0    60   ~ 0
-Changed R8 to 120K\nGives 100 mHz as\nlowest LFO rate
+Changed R8 to 120K\nGives 50 mHz as\nlowest LFO rate
 Text Notes 12500 4375 0    50   ~ 0
 S&H TRI OUT
@@
 P 12725 2475
 F 0 "C2" H 12600 2550 50  0000 L CNN
-F 1 "1000p" H 12450 2350 50  0000 L CNN
+F 1 "1n" H 12600 2350 50  0000 L CNN
 F 2 "MyModules:SM0603-C-JRL" H 12725 2475 60  0001 C CNN
 F 3 "" H 12725 2475 60  0000 C CNN
@@
 	12725 2275 12500 2275
 Connection ~ 12500 2275
-Text Notes 29400 20050 0    200  ~ 40
+Text Notes 31075 21100 0    150  ~ 0
 SYSTEM80 INC. 2017
+Text Notes 32900 21375 0    60   ~ 0
+1.4
+Text Notes 30425 21375 0    60   ~ 0
+1.4
+Text Notes 29375 20675 0    150  ~ 30
+'850' modulation/noise source
+Text Notes 29700 21225 0    60   ~ 0
+LFO, S&H, NOISE, SLEW EURORACK MODULE
 $EndSCHEMATC
